Commit message: add scene for franka panda

File: src/franka_description/robots/hand.xacro (robot description, xacro)
@@ -29,4 +29,6 @@
       <!-- end for simulation -->
     </link>
+    <link name="${ns}_grip_center"/>
+    <joint name="${ns}_grip_center_joint" type="fixed">
     <link name="${ns}_leftfinger">
       <visual>

Commit message: add grip center

File: src/franka_description/robots/hand.xacro (robot description, xacro)
@@ -31,4 +31,8 @@
     <link name="${ns}_grip_center"/>
     <joint name="${ns}_grip_center_joint" type="fixed">
+			<origin xyz="0 0 0.2" rpy="0 0 0" />
+			<parent link="${ns}_hand" />
+			<child link="${ns}_grip_center" />
+		</joint>
     <link name="${ns}_leftfinger">
       <visual>

Commit message: change arm end effector

File: src/franka_description/robots/hand.xacro (robot description, xacro)
@@ -31,5 +31,5 @@
     <link name="${ns}_grip_center"/>
     <joint name="${ns}_grip_center_joint" type="fixed">
-			<origin xyz="0 0 0.2" rpy="0 0 0" />
+			<origin xyz="0 0 0.1" rpy="0 0 0" />
 			<parent link="${ns}_hand" />
 			<child link="${ns}_grip_center" />
