Commit message: add moveit changes for exchanging end effector

File: src/franka_moveit_config/config/gazebo_panda_hand_camera.urdf (robot description, URDF)
Before this commit: robot panda_hand_camera, 15 links, 14 joints
Links:
- added link panda_grip_center
Joints:
- added joint panda_grip_center_joint: type fixed, parent panda_hand, child panda_grip_center, origin xyz=0 0 0.1 rpy=0 0 0
